File: Hardware/ESPRO_2.brd (EAGLE design)
At the start: 120 x 85 mm, 60 parts, among them IC1 AT24CP, P8X32A P8X32A-D40, Q1 5MHz

Commit message: Update Hardware
Routing:
- net N$5: track 16.0 -> 15.1 mm, vias 1 -> 0
- net N$6: track 18.8 -> 18.0 mm, vias 1 -> 0
- net N$50: track 70.1 -> 69.9 mm, vias 3 -> 2
- net P29: vias 10 -> 9
- net P28: vias 8 -> 7
- net P21: vias 6 -> 5
- net P20: vias 5 -> 3
- net P18: vias 4 -> 3
- net N$79: vias 1 -> 0
- net N$19: vias 4 -> 2
- net N$1: vias 2 -> 1
- net E8: vias 1 -> 0
- net E2: vias 4 -> 3

Commit message: Update Hardware
Parts:
- C1: value 2,2µ -> 100nF
Changed lines of the file:
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@@
 <element name="R1" library="rcl" package="0204/7" value="10k" x="3.429" y="19.939" rot="R270"/>
 <element name="R22" library="rcl" package="0204/7" value="10k" x="11.176" y="12.573" rot="R180"/>
-<element name="C1" library="rcl" package="C025-030X050" value="2,2µ" x="10.287" y="32.131" rot="R180"/>
+<element name="C1" library="rcl" package="C025-030X050" value="100nF" x="10.287" y="32.131" rot="R180"/>
 <element name="C2" library="rcl" package="C025-030X050" value="100nF" x="14.986" y="37.465"/>
 <element name="C3" library="rcl" package="E2-4" value="10µ" x="26.162" y="67.564" rot="R90"/>
